Commit message: URDF Loader must have axis xyz defined

File: urdf/galbot_one_golf.urdf (robot description, URDF)
Before this commit: robot galbot_one_golf, 104 links, 103 joints
Joints:
- joint head_end_effector_mount_joint: axis  -> 0 0 1
- joint torso_head_mount_joint: axis  -> 0 0 1
- joint torso_left_arm_mount_joint: axis  -> 0 0 1
- joint torso_right_arm_mount_joint: axis  -> 0 0 1
